Commit message: sompoch update ver03

File: description/gazebo_control.xacro (robot description, xacro)
@@ -18,4 +18,8 @@
             <publish_wheel_tf>true</publish_wheel_tf>
         </plugin>
+        <plugin name="joint_state_publisher" filename="libgazebo_ros_joint_state_publisher.so">
+                <joint_name>caster_wheel_back_joint</joint_name>
+                <joint_name>caster_wheel_front_joint</joint_name>
+        </plugin>
     </gazebo>
 </robot>

File: description/robot_core.xacro (robot description, xacro)
@@ -99,5 +99,5 @@
 </gazebo>
 <joint name="caster_wheel_front_joint" type="continuous">
-    <parent link="base_link"/>
+    <parent link="base_chassis_wheel"/>
     <child link="caster_wheel_front"/>
     <origin xyz="0.12 0 -0.02125"  rpy="0 0 0"/>
@@ -124,5 +124,5 @@
 </gazebo>
 <joint name="caster_wheel_back_joint" type="continuous">
-    <parent link="base_link"/>
+    <parent link="base_chassis_wheel"/>
     <child link="caster_wheel_back"/>
     <origin xyz="-0.12 0 -0.02125" rpy="0 0 0"/>

Commit message: configuration NAV2 success

File: description/gazebo_control.xacro (robot description, xacro)
@@ -18,8 +18,9 @@
             <publish_wheel_tf>true</publish_wheel_tf>
         </plugin>
-        <plugin name="joint_state_publisher" filename="libgazebo_ros_joint_state_publisher.so">
+        <!-- <plugin name="joint_state_publisher" filename="libgazebo_ros_joint_state_publisher.so">
+                <update_rate>20</update_rate>
                 <joint_name>caster_wheel_back_joint</joint_name>
                 <joint_name>caster_wheel_front_joint</joint_name>
-        </plugin>
+        </plugin> -->
     </gazebo>
 </robot>

File: description/robot.urdf.xacro (robot description, xacro)
@@ -1,5 +1,13 @@
 <?xml version="1.0"?>
 <robot xmlns:xacro="http://www.ros.org/wiki/xacro"  name="robot">
-    <xacro:include filename="robot_core.xacro"/>
-    <xacro:include filename="gazebo_control.xacro"/>
+    <xacro:arg name="use_ros2_control" default="true"/>
+    <xacro:arg name="sim_mode" default="false"/>
+    <xacro:include filename="robot_core.xacro" />
+    <xacro:if value="$(arg use_ros2_control)">
+        <xacro:include filename="ros2_control.xacro" />
+    </xacro:if>
+    <xacro:unless value="$(arg use_ros2_control)">
+        <xacro:include filename="gazebo_control.xacro" />
+    </xacro:unless>
+    <xacro:include filename="lidar.xacro" />
 </robot>

File: description/robot_core.xacro (robot description, xacro)
@@ -20,5 +20,15 @@
     <color rgba="0 1 0 1" />
 </material>
+<material name="red">
+    <color rgba="1 0 0 1" />
+</material>
 <link name="base_link">
+</link>
+<joint name="base_footprint_joint" type="fixed">
+    <parent link="base_link"/>
+    <child link="base_footprint"/>
+    <origin xyz="0 0 0" rpy="0 0 0"/>
+</joint>
+<link name="base_footprint">
 </link>
 <joint name="chassis_wheel_joint" type="fixed">

Commit message: Update New BLDC_2025

File: description/gazebo_control.xacro (robot description, xacro)
@@ -6,6 +6,6 @@
             <left_joint>left_wheel_joint</left_joint>
             <right_joint>right_wheel_joint</right_joint>
-            <wheel_separation>0.338</wheel_separation>
-            <wheel_diameter>0.085</wheel_diameter>
+            <wheel_separation>0.4</wheel_separation>
+            <wheel_diameter>0.13</wheel_diameter>
             <!-- Limits -->
             <max_wheel_torque>200</max_wheel_torque>

File: description/lidar.xacro (robot description, xacro)
@@ -4,5 +4,5 @@
         <parent link="Topplate"/>
         <child link="laser_frame"/>
-        <origin xyz="0 0 0.01" rpy="0 0 0"/>
+        <origin xyz="0.145 0 0.01" rpy="0 0 0"/>
     </joint>
     <link name="laser_frame">
@@ -11,5 +11,5 @@
                 <cylinder radius="0.05" length="0.04"/>
             </geometry>
-            <material name="red"/>
+            <material name="black"/>
         </visual>
         <collision>
@@ -23,5 +23,5 @@
     </link>
     <gazebo reference="laser_frame">
-        <material>Gazebo/Red</material>
+        <material>Gazebo/Black</material>
         <sensor name="laser" type="ray">
             <pose> 0 0 0 0 0 0 </pose>
@@ -37,5 +37,5 @@
                 </scan>
                 <range>
-                    <min>0.3</min>
+                    <min>0.45</min>
                     <max>12</max>
                 </range>

File: description/robot_core.xacro (robot description, xacro)
@@ -41,5 +41,5 @@
         <origin xyz="0 0 0" rpy="0 0 0"/>
         <geometry>
-            <cylinder radius="0.15" length="0.02"/>
+            <box size="0.40 0.40 0.02"/>
         </geometry>
         <material name="orange"/>
@@ -48,10 +48,12 @@
         <origin xyz="0 0 0" rpy="0 0 0"/>
         <geometry>
-            <cylinder radius="0.15" length="0.02"/>
-        </geometry>
-    </collision>
-    <xacro:inertial_cylinder mass="0.5" length="0.02" radius="0.15">
-            <origin xyz="0 0 0" rpy="0 0 0"/>
-    </xacro:inertial_cylinder>
+            <box size="0.40 0.40 0.02"/>
+        </geometry>
+    </collision>
+    <inertial>
+        <mass value="0.5"/>
+        <origin xyz="0 0 0" rpy="0 0 0"/>
+        <inertia ixx="0.001" iyy="0.001" izz="0.001" ixy="0.0" ixz="0.0" iyz="0.0"/>
+    </inertial>
 </link>
 <gazebo reference="base_chassis_wheel">
@@ -61,5 +63,5 @@
     <parent link="base_link"/>
     <child link="right_wheel"/>
-    <origin xyz="0 -0.169 0" rpy="1.57 0 0"/>
+    <origin xyz="0 -0.22 0" rpy="1.57 0 0"/>
     <axis xyz="0 0 -1"/>
 </joint>
@@ -67,5 +69,5 @@
     <visual>
         <geometry>
-            <cylinder radius="0.0425" length="0.048"/>
+            <cylinder radius="0.065" length="0.04"/>
         </geometry>
         <material name="green"/>
@@ -73,8 +75,8 @@
     <collision>
         <geometry>
-            <cylinder radius="0.0425" length="0.048"/>
-        </geometry>
-    </collision>
-    <xacro:inertial_cylinder mass="0.1" length="0.048" radius="0.0425">
+            <cylinder radius="0.065" length="0.04"/>
+        </geometry>
+    </collision>
+    <xacro:inertial_cylinder mass="1.95" length="0.04" radius="0.065">
             <origin xyz="0 0 0" rpy="0 0 0"/>
     </xacro:inertial_cylinder>
@@ -86,5 +88,5 @@
     <parent link="base_link"/>
     <child link="left_wheel"/>
-    <origin xyz="0 0.169 0" rpy="-1.57 0 0"/>
+    <origin xyz="0 0.22 0" rpy="-1.57 0 0"/>
     <axis xyz="0 0 1"/>
 </joint>
@@ -92,5 +94,5 @@
     <visual>
         <geometry>
-            <cylinder radius="0.0425" length="0.048"/>
+            <cylinder radius="0.065" length="0.04"/>
         </geometry>
         <material name="green"/>
@@ -98,8 +100,8 @@
     <collision>
         <geometry>
-            <cylinder radius="0.0425" length="0.048"/>
-        </geometry>
-    </collision>
-    <xacro:inertial_cylinder mass="0.1" length="0.048" radius="0.0425">
+            <cylinder radius="0.065" length="0.04"/>
+        </geometry>
+    </collision>
+    <xacro:inertial_cylinder mass="1.95" length="0.04" radius="0.065">
             <origin xyz="0 0 0" rpy="0 0 0"/>
     </xacro:inertial_cylinder>
@@ -111,5 +113,5 @@
     <parent link="base_chassis_wheel"/>
     <child link="caster_wheel_front"/>
-    <origin xyz="0.12 0 -0.02125"  rpy="0 0 0"/>
+    <origin xyz="0.15 0 -0.0325"  rpy="0 0 0"/>
     <axis xyz="0 1 1"/>
 </joint>
@@ -117,14 +119,14 @@
     <visual>
         <geometry>
-            <sphere radius="0.02125"/>
-        </geometry>
-        <material name="white"/>
-    </visual>
-    <collision>
-        <geometry>
-            <sphere radius="0.02125"/>
-        </geometry>
-    </collision>
-    <xacro:inertial_sphere mass="0.1" radius="0.02125">
+            <sphere radius="0.0325"/>
+        </geometry>
+        <material name="white"/>
+    </visual>
+    <collision>
+        <geometry>
+            <sphere radius="0.0325"/>
+        </geometry>
+    </collision>
+    <xacro:inertial_sphere mass="0.2" radius="0.0325">
             <origin xyz="0 0 0" rpy="0 0 0"/>
     </xacro:inertial_sphere>
@@ -136,5 +138,5 @@
     <parent link="base_chassis_wheel"/>
     <child link="caster_wheel_back"/>
-    <origin xyz="-0.12 0 -0.02125" rpy="0 0 0"/>
+    <origin xyz="-0.15 0 -0.0325" rpy="0 0 0"/>
     <axis xyz="0 1 1"/>
 </joint>
@@ -142,14 +144,14 @@
     <visual>
         <geometry>
-            <sphere radius="0.02125"/>
-        </geometry>
-        <material name="white"/>
-    </visual>
-    <collision>
-        <geometry>
-            <sphere radius="0.02125"/>
-        </geometry>
-    </collision>
-    <xacro:inertial_sphere mass="0.1" radius="0.02125">
+            <sphere radius="0.0325"/>
+        </geometry>
+        <material name="white"/>
+    </visual>
+    <collision>
+        <geometry>
+            <sphere radius="0.0325"/>
+        </geometry>
+    </collision>
+    <xacro:inertial_sphere mass="0.2" radius="0.0325">
             <origin xyz="0 0 0" rpy="0 0 0"/>
     </xacro:inertial_sphere>
@@ -161,16 +163,16 @@
     <parent link="base_chassis_wheel"/>
     <child link="columnA"/>
-    <origin xyz="-0.14 0 0.085"/>
+    <origin xyz="-0.17 -0.17 0.21"/>
 </joint>
 <link name="columnA">
     <visual>
         <geometry>
-            <cylinder radius="0.01" length="0.15"/>
-        </geometry>
-        <material name="white"/>
-    </visual>
-    <collision>
-        <geometry>
-            <cylinder radius="0.01" length="0.15"/>
+            <box size="0.03 0.03 0.4"/>
+        </geometry>
+        <material name="white"/>
+    </visual>
+    <collision>
+        <geometry>
+            <box size="0.03 0.03 0.4"/>
         </geometry>
     </collision>
@@ -179,56 +181,84 @@
     <parent link="base_chassis_wheel"/>
     <child link="columnB"/>
-    <origin xyz="0.14 0 0.085"/>
+    <origin xyz="0.17 -0.17 0.21"/>
 </joint>
 <link name="columnB">
     <visual>
         <geometry>
-            <cylinder radius="0.01" length="0.15"/>
-        </geometry>
-        <material name="white"/>
-    </visual>
-    <collision>
-        <geometry>
-            <cylinder radius="0.01" length="0.15"/>
-        </geometry>
-    </collision>
-</link>
+            <box size="0.03 0.03 0.4"/>
+        </geometry>
+        <material name="white"/>
+    </visual>
+    <collision>
+        <geometry>
+            <box size="0.03 0.03 0.4"/>
+        </geometry>
+    </collision>
+</link>
+<joint name="columnC_joint" type="fixed">
+    <parent link="base_chassis_wheel"/>
+    <child link="columnC"/>
+    <origin xyz="-0.17 0.17 0.21"/>
+</joint>
 <link name="columnC">
     <visual>
         <geometry>
-            <cylinder radius="0.01" length="0.15"/>
-        </geometry>
-        <material name="white"/>
-    </visual>
-    <collision>
-        <geometry>
-            <cylinder radius="0.01" length="0.15"/>
-        </geometry>
-    </collision>
-</link>
-<joint name="columnC_joint" type="fixed">
-    <parent link="base_chassis_wheel"/>
-    <child link="columnC"/>
-    <origin xyz="0 -0.14 0.085"/>
-</joint>
+            <box size="0.03 0.03 0.4"/>
+        </geometry>
+        <material name="white"/>
+    </visual>
+    <collision>
+        <geometry>
+            <box size="0.03 0.03 0.4"/>
+        </geometry>
+    </collision>
+</link>
 <joint name="columnD_joint" type="fixed">
     <parent link="base_chassis_wheel"/>
     <child link="columnD"/>
-    <origin xyz="0 0.14 0.085"/>
+    <origin xyz="0.17 0.17 0.21"/>
 </joint>
 <link name="columnD">
     <visual>
         <geometry>
-            <cylinder radius="0.01" length="0.15"/>
-        </geometry>
-        <material name="white"/>
-    </visual>
-    <collision>
-        <geometry>
-            <cylinder radius="0.01" length="0.15"/>
+            <box size="0.03 0.03 0.4"/>
+        </geometry>
+        <material name="white"/>
+    </visual>
+    <collision>
+        <geometry>
+            <box size="0.03 0.03 0.4"/>
         </geometry>
     </collision>
 </link>
 <joint name="plateA_joint" type="fixed">
+    <parent link="base_chassis_wheel"/>
+    <child link="plateA"/>
+    <origin xyz="0 0 0.21"/>
+</joint>
+<link name="plateA">
+    <visual>
+        <origin xyz="0 0 0" rpy="0 0 0"/>
+        <geometry>
+            <box size="0.40 0.40 0.02"/>
+        </geometry>
+        <material name="orange"/>
+    </visual>
+    <collision>
+        <origin xyz="0 0 0" rpy="0 0 0"/>
+        <geometry>
+            <box size="0.40 0.40 0.02"/>
+        </geometry>
+    </collision>
+    <inertial>
+        <mass value="0.5"/>
+        <origin xyz="0 0 0" rpy="0 0 0"/>
+        <inertia ixx="0.001" iyy="0.001" izz="0.001" ixy="0.0" ixz="0.0" iyz="0.0"/>
+    </inertial>
+</link>
+<gazebo reference="plateA">
+    <material>Gazebo/Orange</material>
+</gazebo>
+<!-- <joint name="plateA_joint" type="fixed">
     <parent link="base_chassis_wheel"/>
     <child link="plateA"/>
@@ -250,9 +280,9 @@
             <origin xyz="0 0 0" rpy="0 0 0"/>
     </xacro:inertial_cylinder>
-</link>
-<gazebo reference="plateA">
+</link> -->
+<!-- <gazebo reference="plateA">
     <material>Gazebo/Orange</material>
-</gazebo>
-<joint name="columnG_joint" type="fixed">
+</gazebo> -->
+<!-- <joint name="columnG_joint" type="fixed">
     <parent link="plateA"/>
     <child link="columnG"/>
@@ -295,8 +325,36 @@
 <gazebo reference="columnH">
     <material>Gazebo/White</material>
-</gazebo>
+</gazebo> -->
 <joint name="Topplate_joint" type="fixed">
     <parent link="plateA"/>
     <child link="Topplate"/>
+    <origin xyz="0 0 0.21"/>
+</joint>
+<link name="Topplate">
+    <visual>
+        <origin xyz="0 0 0" rpy="0 0 0"/>
+        <geometry>
+            <box size="0.40 0.40 0.02"/>
+        </geometry>
+        <material name="orange"/>
+    </visual>
+    <collision>
+        <origin xyz="0 0 0" rpy="0 0 0"/>
+        <geometry>
+            <box size="0.40 0.40 0.02"/>
+        </geometry>
+    </collision>
+    <inertial>
+        <mass value="0.5"/>
+        <origin xyz="0 0 0" rpy="0 0 0"/>
+        <inertia ixx="0.001" iyy="0.001" izz="0.001" ixy="0.0" ixz="0.0" iyz="0.0"/>
+    </inertial>
+</link>
+<gazebo reference="Topplate">
+    <material>Gazebo/Orange</material>
+</gazebo>
+<!-- <joint name="Topplate_joint" type="fixed">
+    <parent link="plateA"/>
+    <child link="Topplate"/>
     <origin xyz="0 0 0.155"/>
 </joint>
@@ -319,4 +377,4 @@
 <gazebo reference="Topplate">
     <material>Gazebo/Green</material>
-</gazebo>
+</gazebo> -->
 </robot>
