Commit message: add URDF robot

File: description/robot_core.xacro (robot description, xacro)
@@ -45,4 +45,7 @@
     </xacro:inertial_cylinder>
 </link>
+<gazebo reference="base_chassis_wheel">
+    <material>Gazebo/Orange</material>
+</gazebo>
 <joint name="right_wheel_joint" type="continuous">
     <parent link="base_link"/>
@@ -67,4 +70,7 @@
     </xacro:inertial_cylinder>
 </link>
+<gazebo reference="right_wheel">
+    <material>Gazebo/Green</material>
+</gazebo>
 <joint name="left_wheel_joint" type="continuous">
     <parent link="base_link"/>
@@ -89,46 +95,57 @@
     </xacro:inertial_cylinder>
 </link>
-<joint name="caster_wheel_front_joint" type="fixed">
-    <parent link="base_chassis_wheel"/>
+<gazebo reference="left_wheel">
+    <material>Gazebo/Green</material>
+</gazebo>
+<joint name="caster_wheel_front_joint" type="continuous">
+    <parent link="base_link"/>
     <child link="caster_wheel_front"/>
-    <origin xyz="0.12 0 -0.02"/>
+    <origin xyz="0.12 0 -0.02125"  rpy="0 0 0"/>
+    <axis xyz="0 1 1"/>
 </joint>
 <link name="caster_wheel_front">
     <visual>
         <geometry>
-            <sphere radius="0.03"/>
-        </geometry>
-        <material name="white"/>
-    </visual>
-    <collision>
-        <geometry>
-            <sphere radius="0.03"/>
-        </geometry>
-    </collision>
-    <xacro:inertial_sphere mass="0.1" radius="0.03">
-            <origin xyz="0 0 0" rpy="0 0 0"/>
-        </xacro:inertial_sphere>
-</link>
-<joint name="caster_wheel_back_joint" type="fixed">
-    <parent link="base_chassis_wheel"/>
+            <sphere radius="0.02125"/>
+        </geometry>
+        <material name="white"/>
+    </visual>
+    <collision>
+        <geometry>
+            <sphere radius="0.02125"/>
+        </geometry>
+    </collision>
+    <xacro:inertial_sphere mass="0.1" radius="0.02125">
+            <origin xyz="0 0 0" rpy="0 0 0"/>
+    </xacro:inertial_sphere>
+</link>
+<gazebo reference="caster_wheel_front">
+    <material>Gazebo/White</material>
+</gazebo>
+<joint name="caster_wheel_back_joint" type="continuous">
+    <parent link="base_link"/>
     <child link="caster_wheel_back"/>
-    <origin xyz="-0.12 0 -0.02"/>
+    <origin xyz="-0.12 0 -0.02125" rpy="0 0 0"/>
+    <axis xyz="0 1 1"/>
 </joint>
 <link name="caster_wheel_back">
     <visual>
         <geometry>
-            <sphere radius="0.03"/>
-        </geometry>
-        <material name="white"/>
-    </visual>
-    <collision>
-        <geometry>
-            <sphere radius="0.03"/>
-        </geometry>
-    </collision>
-    <xacro:inertial_sphere mass="0.1" radius="0.03">
+            <sphere radius="0.02125"/>
+        </geometry>
+        <material name="white"/>
+    </visual>
+    <collision>
+        <geometry>
+            <sphere radius="0.02125"/>
+        </geometry>
+    </collision>
+    <xacro:inertial_sphere mass="0.1" radius="0.02125">
             <origin xyz="0 0 0" rpy="0 0 0"/>
     </xacro:inertial_sphere>
 </link>
+<gazebo reference="caster_wheel_back">
+    <material>Gazebo/White</material>
+</gazebo>
 <joint name="columnA_joint" type="fixed">
     <parent link="base_chassis_wheel"/>
@@ -224,4 +241,7 @@
     </xacro:inertial_cylinder>
 </link>
+<gazebo reference="plateA">
+    <material>Gazebo/Orange</material>
+</gazebo>
 <joint name="columnG_joint" type="fixed">
     <parent link="plateA"/>
@@ -242,4 +262,7 @@
     </collision>
 </link>
+<gazebo reference="columnG">
+    <material>Gazebo/White</material>
+</gazebo>
 <joint name="columnH_joint" type="fixed">
     <parent link="plateA"/>
@@ -260,4 +283,7 @@
     </collision>
 </link>
+<gazebo reference="columnH">
+    <material>Gazebo/White</material>
+</gazebo>
 <joint name="Topplate_joint" type="fixed">
     <parent link="plateA"/>
@@ -281,3 +307,6 @@
     </xacro:inertial_cylinder>
 </link>
+<gazebo reference="Topplate">
+    <material>Gazebo/Green</material>
+</gazebo>
 </robot>

Commit message: Update from Rp4 to git 30_06_2025

File: description/robot_core.xacro (robot description, xacro)
@@ -110,5 +110,5 @@
     <material>Gazebo/Green</material>
 </gazebo>
-<joint name="caster_wheel_front_joint" type="continuous">
+<joint name="caster_wheel_front_joint" type="fixed">
     <parent link="base_chassis_wheel"/>
     <child link="caster_wheel_front"/>
@@ -135,5 +135,5 @@
     <material>Gazebo/White</material>
 </gazebo>
-<joint name="caster_wheel_back_joint" type="continuous">
+<joint name="caster_wheel_back_joint" type="fixed">
     <parent link="base_chassis_wheel"/>
     <child link="caster_wheel_back"/>

File: description/ros2_control.xacro (robot description, xacro)
@@ -9,5 +9,5 @@
                 <param name="loop_rate">30</param>
                 <param name="device">/dev/ttyUSB0</param>
-                <param name="baud_rate">57600</param>
+                <param name="baud_rate">115200</param>
                 <param name="timeout">1000</param>
                 <param name="enc_counts_per_rev">4096</param>
@@ -15,6 +15,6 @@
             <joint name="left_wheel_joint">
                 <command_interface name="velocity">
-                    <param name="min">-10</param>
-                    <param name="max">10</param>
+                    <param name="min">-1</param>
+                    <param name="max">1</param>
                 </command_interface>
                 <state_interface name="velocity"/>
@@ -23,6 +23,6 @@
             <joint name="right_wheel_joint">
                 <command_interface name="velocity">
-                    <param name="min">-10</param>
-                    <param name="max">10</param>
+                    <param name="min">-1</param>
+                    <param name="max">1</param>
                 </command_interface>
                 <state_interface name="velocity"/>
